File: KeyboardProject.kicad_pcb (KiCad board)
At the start: 2 copper layers, 323.8 x 133.4 mm, 157 parts, among them SW1 SW_Push, SW10 SW_Push, SW11 SW_Push, SW12 SW_Push, SW13 SW_Push, SW14 SW_Push, SW15 SW_Push, SW16 SW_Push, SW17 SW_Push, SW18 SW_Push, SW19 SW_Push, SW2 SW_Push, SW20 SW_Push, SW21 SW_Push, SW22 SW_Push, SW23 SW_Push, SW24 SW_Push, SW25 SW_Push, SW26 SW_Push, SW27 SW_Push, SW28 SW_Push, SW29 SW_Push, SW3 SW_Push, SW30 SW_Push, SW31 SW_Push, SW32 SW_Push, SW33 SW_Push, SW34 SW_Push, SW35 SW_Push, SW36 SW_Push, SW37 SW_Push, SW38 SW_Push, SW39 SW_Push, SW4 SW_Push, SW40 SW_Push, SW41 SW_Push, SW42 SW_Push, SW43 SW_Push, SW44 SW_Push, SW45 SW_Push, SW46 SW_Push, SW47 SW_Push, SW48 SW_Push, SW49 SW_Push, SW5 SW_Push, SW50 SW_Push, SW51 SW_Push, SW52 SW_Push, SW53 SW_Push, SW54 SW_Push, SW55 SW_Push, SW56 SW_Push, SW57 SW_Push, SW58 SW_Push, SW59 SW_Push, SW6 SW_Push, SW60 SW_Push, SW61 SW_Push, SW62 SW_Push, SW63 SW_Push, SW64 SW_Push, SW65 SW_Push, SW66 SW_Push, SW67 SW_Push, SW68 SW_Push, SW69 SW_Push, SW7 SW_Push, SW70 SW_Push, SW71 SW_Push, SW72 SW_Push, SW73 SW_Push, SW74 SW_Push, SW75 SW_Push, SW76 SW_Push, SW77 SW_Push, SW8 SW_Push, SW82 Rotary_Encoder_Switch, SW9 SW_Push, U1 Teensy4.0

Commit message: Save progress
Parts:
- removed SW1, SW10, SW11, SW12, SW13, SW14, SW15, SW16, SW17, SW18, SW19, SW2, SW20, SW21, SW22, SW24, SW25, SW26, SW27, SW28, SW29, SW30, SW31, SW32, SW33, SW34, SW35, SW36, SW37, SW38, SW40, SW41, SW42, SW43, SW44, SW45, SW46, SW47, SW48, SW49, SW50, SW51, SW52, SW53, SW54, SW56, SW57, SW58, SW59, SW6, SW60, SW62, SW63, SW64, SW65, SW66, SW67, SW68, SW69, SW7, SW70, SW72, SW76, SW77, SW8, SW9: SW_Push, Button_Switch_Keyboard:SW_Cherry_MX_1.00u_PCB
- removed SW23, SW55, SW61: SW_Push, Button_Switch_Keyboard:SW_Cherry_MX_1.25u_PCB
- removed SW3, SW74: SW_Push, Button_Switch_Keyboard:SW_Cherry_MX_1.50u_PCB
- removed SW39: SW_Push, Button_Switch_Keyboard:SW_Cherry_MX_6.25u_PCB
- removed SW4, SW71: SW_Push, Button_Switch_Keyboard:SW_Cherry_MX_1.75u_PCB
- removed SW5, SW73: SW_Push, Button_Switch_Keyboard:SW_Cherry_MX_2.00u_PCB
- removed SW75: SW_Push, Button_Switch_Keyboard:SW_Cherry_MX_2.25u_PCB
- added A1: SW_Push, Button_Switch_Keyboard:SW_Cherry_MX_1.00u_PCB, F.Cu at (52.5, -64.6)
- added B1: SW_Push, Button_Switch_Keyboard:SW_Cherry_MX_1.00u_PCB, F.Cu at (138.3, -45.6)
- added Backspace1: SW_Push, Button_Switch_Keyboard:SW_Cherry_MX_2.00u_PCB, F.Cu at (276.4, -102.7)
- added C1: SW_Push, Button_Switch_Keyboard:SW_Cherry_MX_1.00u_PCB, F.Cu at (100.2, -45.6)
- added CBrace1: SW_Push, Button_Switch_Keyboard:SW_Cherry_MX_1.00u_PCB, F.Cu at (257.3, -83.7)
- added Caps1: SW_Push, Button_Switch_Keyboard:SW_Cherry_MX_1.75u_PCB, F.Cu at (26.4, -64.6)
- added Comma1: SW_Push, Button_Switch_Keyboard:SW_Cherry_MX_1.00u_PCB, F.Cu at (195.4, -45.6)
- added D79: SW_Push, Button_Switch_Keyboard:SW_Cherry_MX_1.00u_PCB, F.Cu at (90.6, -64.6)
- added DArrow1: SW_Push, Button_Switch_Keyboard:SW_Cherry_MX_1.00u_PCB, F.Cu at (290.7, -21.7)
- added Dash1: SW_Push, Button_Switch_Keyboard:SW_Cherry_MX_1.00u_PCB, F.Cu at (228.8, -102.7)
- added E1: SW_Push, Button_Switch_Keyboard:SW_Cherry_MX_1.00u_PCB, F.Cu at (85.9, -83.7)
- added Eight1: SW_Push, Button_Switch_Keyboard:SW_Cherry_MX_1.00u_PCB, F.Cu at (171.6, -102.7)
- added Enter1: SW_Push, Button_Switch_Keyboard:SW_Cherry_MX_2.25u_PCB, F.Cu at (274.0, -64.6)
- added Esc1: SW_Push, Button_Switch_Keyboard:SW_Cherry_MX_1.00u_PCB, F.Cu at (19.2, -126.5)
- added F1: SW_Push, Button_Switch_Keyboard:SW_Cherry_MX_1.00u_PCB, F.Cu at (47.8, -126.5)
- added F10: SW_Push, Button_Switch_Keyboard:SW_Cherry_MX_1.00u_PCB, F.Cu at (247.8, -126.5)
- added F11: SW_Push, Button_Switch_Keyboard:SW_Cherry_MX_1.00u_PCB, F.Cu at (266.9, -126.5)
- added F12: SW_Push, Button_Switch_Keyboard:SW_Cherry_MX_1.00u_PCB, F.Cu at (285.9, -126.5)
- added F13: SW_Push, Button_Switch_Keyboard:SW_Cherry_MX_1.00u_PCB, F.Cu at (109.7, -64.6)
- added F2: SW_Push, Button_Switch_Keyboard:SW_Cherry_MX_1.00u_PCB, F.Cu at (66.8, -126.5)
- added F3: SW_Push, Button_Switch_Keyboard:SW_Cherry_MX_1.00u_PCB, F.Cu at (85.9, -126.5)
- added F4: SW_Push, Button_Switch_Keyboard:SW_Cherry_MX_1.00u_PCB, F.Cu at (104.9, -126.5)
- added F5: SW_Push, Button_Switch_Keyboard:SW_Cherry_MX_1.00u_PCB, F.Cu at (138.3, -126.5)
- added F6: SW_Push, Button_Switch_Keyboard:SW_Cherry_MX_1.00u_PCB, F.Cu at (157.3, -126.5)
- added F7: SW_Push, Button_Switch_Keyboard:SW_Cherry_MX_1.00u_PCB, F.Cu at (176.4, -126.5)
- added F8: SW_Push, Button_Switch_Keyboard:SW_Cherry_MX_1.00u_PCB, F.Cu at (195.4, -126.5)
- added F9: SW_Push, Button_Switch_Keyboard:SW_Cherry_MX_1.00u_PCB, F.Cu at (228.8, -126.5)
- added Five1: SW_Push, Button_Switch_Keyboard:SW_Cherry_MX_1.00u_PCB, F.Cu at (114.5, -102.7)
- added Fn1: SW_Push, Button_Switch_Keyboard:SW_Cherry_MX_1.00u_PCB, F.Cu at (19.2, -26.5)
- added Four1: SW_Push, Button_Switch_Keyboard:SW_Cherry_MX_1.00u_PCB, F.Cu at (95.4, -102.7)
- added G1: SW_Push, Button_Switch_Keyboard:SW_Cherry_MX_1.00u_PCB, F.Cu at (128.7, -64.6)
- added H1: SW_Push, Button_Switch_Keyboard:SW_Cherry_MX_1.00u_PCB, F.Cu at (147.8, -64.6)
- added I1: SW_Push, Button_Switch_Keyboard:SW_Cherry_MX_1.00u_PCB, F.Cu at (181.1, -83.7)
- added J1: SW_Push, Button_Switch_Keyboard:SW_Cherry_MX_1.00u_PCB, F.Cu at (166.8, -64.6)
- added K1: SW_Push, Button_Switch_Keyboard:SW_Cherry_MX_1.00u_PCB, F.Cu at (185.9, -64.6)
- added L1: SW_Push, Button_Switch_Keyboard:SW_Cherry_MX_1.00u_PCB, F.Cu at (204.9, -64.6)
- added LArrow1: SW_Push, Button_Switch_Keyboard:SW_Cherry_MX_1.00u_PCB, F.Cu at (271.6, -21.7)
- added LCmd1: SW_Push, Button_Switch_Keyboard:SW_Cherry_MX_1.25u_PCB, F.Cu at (78.7, -26.5)
- added LCtrl1: SW_Push, Button_Switch_Keyboard:SW_Cherry_MX_1.00u_PCB, F.Cu at (38.3, -26.5)
- added LOption1: SW_Push, Button_Switch_Keyboard:SW_Cherry_MX_1.00u_PCB, F.Cu at (57.3, -26.5)
- added M1: SW_Push, Button_Switch_Keyboard:SW_Cherry_MX_1.00u_PCB, F.Cu at (176.4, -45.6)
- added N1: SW_Push, Button_Switch_Keyboard:SW_Cherry_MX_1.00u_PCB, F.Cu at (157.3, -45.6)
- added Nine1: SW_Push, Button_Switch_Keyboard:SW_Cherry_MX_1.00u_PCB, F.Cu at (190.7, -102.7)
- added O1: SW_Push, Button_Switch_Keyboard:SW_Cherry_MX_1.00u_PCB, F.Cu at (200.2, -83.7)
- added OBrace1: SW_Push, Button_Switch_Keyboard:SW_Cherry_MX_1.00u_PCB, F.Cu at (238.3, -83.7)
- added One1: SW_Push, Button_Switch_Keyboard:SW_Cherry_MX_1.00u_PCB, F.Cu at (38.3, -102.7)
- added P1: SW_Push, Button_Switch_Keyboard:SW_Cherry_MX_1.00u_PCB, F.Cu at (219.2, -83.7)
- added Period1: SW_Push, Button_Switch_Keyboard:SW_Cherry_MX_1.00u_PCB, F.Cu at (214.5, -45.6)
- added Plus1: SW_Push, Button_Switch_Keyboard:SW_Cherry_MX_1.00u_PCB, F.Cu at (247.8, -102.7)
- added Q1: SW_Push, Button_Switch_Keyboard:SW_Cherry_MX_1.00u_PCB, F.Cu at (47.8, -83.7)
- added QuestionMark1: SW_Push, Button_Switch_Keyboard:SW_Cherry_MX_1.00u_PCB, F.Cu at (233.5, -45.6)
- added Quote1: SW_Push, Button_Switch_Keyboard:SW_Cherry_MX_1.00u_PCB, F.Cu at (243.0, -64.6)
- added R1: SW_Push, Button_Switch_Keyboard:SW_Cherry_MX_1.00u_PCB, F.Cu at (104.9, -83.7)
- added RArrow1: SW_Push, Button_Switch_Keyboard:SW_Cherry_MX_1.00u_PCB, F.Cu at (309.7, -21.7)
- added RCmd1: SW_Push, Button_Switch_Keyboard:SW_Cherry_MX_1.25u_PCB, F.Cu at (221.6, -26.5)
- added ROption1: SW_Push, Button_Switch_Keyboard:SW_Cherry_MX_1.25u_PCB, F.Cu at (245.4, -26.5)
- added S1: SW_Push, Button_Switch_Keyboard:SW_Cherry_MX_1.00u_PCB, F.Cu at (71.6, -64.6)
- added Semi1: SW_Push, Button_Switch_Keyboard:SW_Cherry_MX_1.00u_PCB, F.Cu at (224.0, -64.6)
- added Seven1: SW_Push, Button_Switch_Keyboard:SW_Cherry_MX_1.00u_PCB, F.Cu at (152.6, -102.7)
- added Shift1: SW_Push, Button_Switch_Keyboard:SW_Cherry_MX_2.00u_PCB, F.Cu at (31.1, -45.6)
- added ShiftR1: SW_Push, Button_Switch_Keyboard:SW_Cherry_MX_1.75u_PCB, F.Cu at (259.7, -45.6)
- added Six1: SW_Push, Button_Switch_Keyboard:SW_Cherry_MX_1.00u_PCB, F.Cu at (133.5, -102.7)
- added Slash1: SW_Push, Button_Switch_Keyboard:SW_Cherry_MX_1.50u_PCB, F.Cu at (281.1, -83.7)
- added Space1: SW_Push, Button_Switch_Keyboard:SW_Cherry_MX_6.25u_PCB, F.Cu at (150.2, -26.5)
- added T1: SW_Push, Button_Switch_Keyboard:SW_Cherry_MX_1.00u_PCB, F.Cu at (124.0, -83.7)
- added Tab1: SW_Push, Button_Switch_Keyboard:SW_Cherry_MX_1.50u_PCB, F.Cu at (24.0, -83.7)
- added Three1: SW_Push, Button_Switch_Keyboard:SW_Cherry_MX_1.00u_PCB, F.Cu at (76.4, -102.7)
- added Tilde1: SW_Push, Button_Switch_Keyboard:SW_Cherry_MX_1.00u_PCB, F.Cu at (19.2, -102.7)
- added Two1: SW_Push, Button_Switch_Keyboard:SW_Cherry_MX_1.00u_PCB, F.Cu at (57.3, -102.7)
- added U2: SW_Push, Button_Switch_Keyboard:SW_Cherry_MX_1.00u_PCB, F.Cu at (162.1, -83.7)
- added UArrow1: SW_Push, Button_Switch_Keyboard:SW_Cherry_MX_1.00u_PCB, F.Cu at (290.7, -40.8)
- added V1: SW_Push, Button_Switch_Keyboard:SW_Cherry_MX_1.00u_PCB, F.Cu at (119.2, -45.6)
- added W1: SW_Push, Button_Switch_Keyboard:SW_Cherry_MX_1.00u_PCB, F.Cu at (66.8, -83.7)
- added X1: SW_Push, Button_Switch_Keyboard:SW_Cherry_MX_1.00u_PCB, F.Cu at (81.1, -45.6)
- added Y1: SW_Push, Button_Switch_Keyboard:SW_Cherry_MX_1.00u_PCB, F.Cu at (143.0, -83.7)
- added Z1: SW_Push, Button_Switch_Keyboard:SW_Cherry_MX_1.00u_PCB, F.Cu at (62.1, -45.6)
- added Zero1: SW_Push, Button_Switch_Keyboard:SW_Cherry_MX_1.00u_PCB, F.Cu at (209.7, -102.7)
- D1, D10, D11, D12, D13, D14, D15, D16, D17, D18, D19, D2, D20, D21, D22, D23, D24, D25, D26, D27, D28, D29, D3, D30, D31, D32, D33, D34, D35, D36, D37, D38, D39, D4, D40, D41, D42, D43, D44, D45, D46, D47, D48, D49, D5, D50, D51, D52, D53, D54, D55, D56, D57, D58, D59, D6, D60, D61, D62, D63, D64, D65, D66, D67, D68, D69, D7, D70, D71, D72, D73, D74, D75, D76, D77, D78, D8, D9: value 1N4148 -> 1N4148W; footprint Diode_THT:D_DO-35_SOD27_P7.62mm_Horizontal -> 1n4148-g:DO-35
- moved D76 176.2 mm to (250.0, -64.3), turned to 90 degrees
- moved D77 174.7 mm to (278.6, -42.9), turned to 90 degrees
- moved D74 168.7 mm to (254.8, -102.4), turned to 90 degrees
- moved D75 166.7 mm to (266.7, -83.3), turned to 90 degrees
- moved D68 161.7 mm to (273.8, -121.4), turned to 270 degrees
- moved D1 155.2 mm to (26.2, -121.4), turned to 270 degrees
- moved D12 155.2 mm to (54.8, -121.4), turned to 270 degrees
- moved D18 155.2 mm to (73.8, -121.4), turned to 270 degrees
- moved D24 155.2 mm to (92.9, -121.4), turned to 270 degrees
- moved D29 155.2 mm to (126.2, -121.4), turned to 270 degrees
- moved D34 155.2 mm to (145.3, -121.4), turned to 270 degrees
- moved D40 155.2 mm to (164.3, -121.4), turned to 270 degrees
- moved D45 155.2 mm to (183.4, -121.4), turned to 270 degrees
- moved D50 155.2 mm to (216.7, -121.4), turned to 270 degrees
- moved D56 155.2 mm to (235.7, -121.4), turned to 270 degrees
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Connections:
- net GND renamed /GND
- D73 pad 2: Net-(D73-Pad2) -> /RotarySwitchOut
- D78 pad 2: /RotarySwitchOut -> Net-(D78-Pad2)
- U1 pad 1: Net-(U1-Pad1) -> (no net)
- U1 pad 15: Net-(U1-Pad15) -> (no net)
- U1 pad 16: Net-(U1-Pad16) -> (no net)
- U1 pad 17: Net-(U1-Pad17) -> (no net)
- U1 pad 18: Net-(U1-Pad18) -> (no net)
- U1 pad 19: Net-(U1-Pad19) -> (no net)
- U1 pad 20: Net-(U1-Pad20) -> (no net)
- U1 pad 28: Net-(U1-Pad28) -> (no net)
- U1 pad 31: Net-(U1-Pad31) -> (no net)
- U1 pad 33: Net-(U1-Pad33) -> (no net)
- U1 pad 34: Net-(U1-Pad34) -> (no net)
Routing:
- net /C0: track 496.2 -> 97.5 mm
- net /C1: track 428.8 -> 113.4 mm
- net /C2: track 406.1 -> 107.8 mm
- net /C3: track 384.2 -> 108.0 mm
- net /C4: track 337.8 -> 85.6 mm
- net /C5: track 313.1 -> 97.9 mm
- net /C7: track 295.6 -> 94.6 mm
- net /C6: track 312.9 -> 123.2 mm
- net /C8: track 267.7 -> 96.4 mm
- net /C9: track 318.3 -> 150.9 mm
- net /C11: track 320.5 -> 155.0 mm
- net /C10: track 297.9 -> 154.2 mm
- net /C12: track 243.7 -> 146.9 mm
- net /C13: track 240.2 -> 156.5 mm
- net /R1: track 341.1 -> 289.5 mm
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Other:
- board size 323.8 x 133.4 mm -> 311.9 x 123.8 mm
